Commit message: Update piper_description_d435.urdf

File: src/curobo/content/assets/robot/piper_description/piper_description_d435.urdf (robot description, URDF)
Before this commit: robot piper, 14 links, 13 joints
Joints:
- joint joint7: axis 0 0 1 -> 0 1 0; limit lower=0 upper=0.09 effort=10 velocity=1 -> lower=-0.09 upper=0.0 effort=10 velocity=1; origin xyz=0 0 0.1358 rpy=1.5708 0 0 -> xyz=0 0 0.1358 rpy=0 0 0
